File: ESP32-S3-Breakout.kicad_pcb (KiCad board)
At the start: 4 copper layers, 29 x 54.4 mm, 34 parts, among them J1 USB_C_Receptacle_USB2.0, J2 USB_C_Receptacle_USB2.0, J3 Conn_01x21, J4 Conn_01x21, Q1 Q_NPN_BCE, Q2 Q_NPN_BCE, SW1 SW_Push, SW2 SW_Push, U1 USBLC6-2SC6, U2 USBLC6-2SC6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

Commit message: started 2-layer
Parts:
- J3, J4: moved to F.Cu
- SW1: value SW_Push -> Reset
- SW2: value SW_Push -> Boot
- moved J4 76.1 mm to (167.9, 38.9), turned to 0 degrees
- moved FB2 75.2 mm to (138.4, 66.3), turned to -90 degrees
- moved D2 74.9 mm to (135.1, 66.5)
- moved SW1 72.6 mm to (148.4, 71.9), turned to 0 degrees
- moved U1 67.8 mm to (140.5, 79.4)
- moved J2 67.8 mm to (140.3, 87.9)
- moved C9 67.0 mm to (137.7, 70.6), turned to -90 degrees
- moved R5 66.9 mm to (140.0, 70.9)
- moved R6 65.3 mm to (132.6, 66.6)
- moved SW2 64.1 mm to (136.6, 75.2)
- moved R7 59.8 mm to (132.6, 70.4)
- moved U3 58.8 mm to (129.4, 43.9)
- moved Q2 58.2 mm to (136.3, 79.8), turned to 180 degrees
- moved C1 57.6 mm to (135.1, 70.5)
- moved FB1 57.5 mm to (129.0, 66.5), turned to 0 degrees
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Routing:
- net /EN: track 52.0 -> 0.00 mm, vias 4 -> 0
- net GND: track 42.0 -> 0.00 mm, vias 13 -> 0
- net /IO12: track 33.2 -> 0.00 mm, vias 1 -> 0
- net /IO0: track 31.6 -> 0.00 mm, vias 3 -> 0
- net /TXD0: track 31.1 -> 0.00 mm, vias 2 -> 0
- net /RXD0: track 30.5 -> 0.00 mm, vias 2 -> 0
- net /IO13: track 29.3 -> 0.00 mm, vias 1 -> 0
- net /IO19: track 27.6 -> 0.00 mm, vias 1 -> 0
- net /IO11: track 27.4 -> 0.00 mm, vias 1 -> 0
- net /IO14: track 26.7 -> 0.00 mm, vias 1 -> 0
- net /IO10: track 24.5 -> 0.00 mm, vias 1 -> 0
- net /IO21: track 23.8 -> 0.00 mm, vias 1 -> 0
- net /IO20: track 22.6 -> 0.00 mm, vias 1 -> 0
- net /IO9: track 22.2 -> 0.00 mm, vias 1 -> 0
- net /IO47: track 19.7 -> 0.00 mm, vias 1 -> 0
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- removed copper zone on F.Cu, net +3V3
- removed copper zone on In2.Cu, net +3V3
- removed copper zone on B.Cu, net +5V
- removed copper zone on In1.Cu, net GND
Other:
- board outline removed
- board text removed: "3V3"
- board text removed: "5V"
- board text removed: "EN"
- board text removed: "ESP32-S3 DEV Module"
- board text removed: "GND"
- board text removed: "IO0"
- board text removed: "IO1"
- board text removed: "IO10"
- board text removed: "IO11"
- board text removed: "IO12"
- board text removed: "IO13"
- board text removed: "IO14"
- board text removed: "IO15"
- board text removed: "IO16"
- board text removed: "IO17"
- board text removed: "IO18"
- board text removed: "IO19"
- board text removed: "IO2"
- board text removed: "IO20"
- board text removed: "IO21"
- board text removed: "IO3"
- board text removed: "IO35"
- board text removed: "IO36"
- board text removed: "IO37"
- board text removed: "IO38"
- board text removed: "IO39"
- board text removed: "IO4"
- board text removed: "IO40"
- board text removed: "IO41"
- board text removed: "IO42"
- board text removed: "IO45"
- board text removed: "IO46"
- board text removed: "IO47"
- board text removed: "IO48"
- board text removed: "IO5"
- board text removed: "IO6"
- board text removed: "IO7"
- board text removed: "IO8"
- board text removed: "IO9"
- board text removed: "RXD0"
- board text removed: "Rev 1 12/2022"
- board text removed: "TXD0"
- board text removed: "UART"
- board text removed: "USB"
